Commit message: Adding dummy inertia values to CX165L urdf

File: khi_cx_description/urdf/cx165l_macro.xacro (robot description, xacro)
@@ -40,4 +40,11 @@
     <xacro:property name="j5_velocity_limit" value="${radians(180)}"/>
     <xacro:property name="j6_velocity_limit" value="${radians(280)}"/>
+    <!-- link inertial(TODO : set correct link inertial )-->
+    <xacro:macro name="default_inertial" params="mass">
+      <inertial>
+        <mass value="${mass}" />
+        <inertia ixx="1.0" ixy="0.0" ixz="0.0" iyy="1.0" iyz="0.0" izz="1.0" />
+      </inertial>
+    </xacro:macro>
     <!-- Link 0 -->
     <link name="${prefix}base_link">
@@ -65,4 +72,5 @@
             </geometry>
         </collision>
+        <xacro:default_inertial mass="${j0_mass}"/>
     </link>
     <!-- Link 1 -->
@@ -99,4 +107,5 @@
             </geometry>
         </collision>
+        <xacro:default_inertial mass="${j1_mass}"/>
     </link>
     <!-- Link 2 -->
@@ -133,4 +142,5 @@
             </geometry>
         </collision>
+        <xacro:default_inertial mass="${j2_mass}"/>
     </link>
     <!-- Link 3 -->
@@ -167,4 +177,5 @@
             </geometry>
         </collision>
+        <xacro:default_inertial mass="${j3_mass}"/>
     </link>
     <!-- Link 4 -->
@@ -201,4 +212,5 @@
             </geometry>
         </collision>
+        <xacro:default_inertial mass="${j4_mass}"/>
     </link>
     <!-- Link 5 -->
@@ -235,4 +247,5 @@
             </geometry>
         </collision>
+        <xacro:default_inertial mass="${j5_mass}"/>
     </link>
     <!-- Link 6 -->
@@ -269,4 +282,5 @@
             </geometry>
         </collision>
+        <xacro:default_inertial mass="${j6_mass}"/>
     </link>
   </xacro:macro>
