Commit message: Added ISU Lab environment & MoveIt Config Pkg
Added ISU lab environment urdf xacro including base plate, walls, and floor. 
Added PushCorp adapter, complaint tool, and robot to the end of joint 6. 
Added convex hull STL files to simplify joint collision. 
Fixed robot urdf orientation translation issue from SOLIDWORKS.
Created MoveIt Config package - needs additional work.

File: khi_cx_description/urdf/cx165l.urdf.xacro (robot description, xacro)
@@ -8,5 +8,5 @@
   <joint name="world2base" type="fixed">
     <parent link="world"/>
-    <child link="base_link"/>
+    <child link="base_plate"/>
     <origin rpy="0 0 0" xyz="0 0 0"/>
   </joint>

File: khi_cx_description/urdf/cx165l_macro.xacro (robot description, xacro)
@@ -2,6 +2,7 @@
 <robot xmlns:xacro="http://ros.org/wiki/xacro">
   <xacro:macro name="khi_cx165l" params="prefix">
-    <xacro:include filename="$(find khi_rs_description)/urdf/rs.transmission.xacro" />
-    <xacro:include filename="$(find khi_rs_description)/urdf/common.gazebo.xacro" />
+    <xacro:include filename="$(find khi_cx_description)/urdf/cx.transmission.xacro" />
+    <xacro:include filename="$(find khi_cx_description)/urdf/common.gazebo.xacro" />
+    <xacro:include filename="$(find khi_cx_description)/urdf/isu_lab.xacro" />
     <!-- link rviz colors -->
     <material name="White">
@@ -44,7 +45,12 @@
       <inertial>
         <mass value="${mass}" />
-        <inertia ixx="1.0" ixy="0.0" ixz="0.0" iyy="1.0" iyz="0.0" izz="1.0" />
+        <inertia ixx="0.1" ixy="0.0" ixz="0.0" iyy="0.1" iyz="0.0" izz="0.1" />
       </inertial>
     </xacro:macro>
+    <joint name="${prefix}base_link_joint" type="fixed">
+        <parent link="base_plate" />
+        <child link="base_link" />
+        <origin rpy="0 0 0" xyz="0 0 0" />
+    </joint>
     <!-- Link 0 -->
     <link name="${prefix}base_link">
@@ -55,19 +61,19 @@
             <geometry>
                 <mesh
-                filename="package://khi_cx_description/meshes/CX165L-BC01_BASE.STL" />
-            </geometry>
-            <material
-                name="">
-                <color
-                rgba="0.75294 0.75294 0.75294 1" />
-            </material>
-        </visual>
-        <collision>
-            <origin
-                xyz="0 0 0"
-                rpy="0 0 0" />
-            <geometry>
-                <mesh
-                filename="package://khi_cx_description/meshes/CX165L-BC01_BASE.STL" />
+                filename="package://khi_cx_description/meshes/CX165L-BASE.STL" />
+            </geometry>
+            <material
+                name="">
+                <color
+                rgba="0.75294 0.75294 0.75294 1" />
+            </material>
+        </visual>
+        <collision>
+            <origin
+                xyz="0 0 0"
+                rpy="0 0 0" />
+            <geometry>
+                <mesh
+                filename="package://khi_cx_description/meshes/CX165L-BASE-HULL.STL" />
             </geometry>
         </collision>
@@ -78,5 +84,5 @@
       <axis xyz="0 0 -1" rpy="0 0 0" />
       <limit effort="1000.0" lower="${j1_lower_limit}" upper="${j1_upper_limit}" velocity="${j1_velocity_limit}"/>
-      <origin xyz="0 -1.7415 0.051743" rpy="-0.0087266 0 0" />
+      <origin xyz="0 0 0.55" rpy="0 0 0" />
       <parent link="${prefix}base_link"/>
       <child link="${prefix}link1"/>
@@ -90,19 +96,19 @@
             <geometry>
                 <mesh
-                filename="package://khi_cx_description/meshes/CX165L-BC01_J1.STL"/>
-            </geometry>
-            <material
-                name="">
-                <color
-                rgba="0.75294 0.75294 0.75294 1" />
-            </material>
-        </visual>
-        <collision>
-            <origin
-                xyz="0 0 0"
-                rpy="0 0 0" />
-            <geometry>
-                <mesh
-                filename="package://khi_cx_description/meshes/CX165L-BC01_J1.STL" />
+                filename="package://khi_cx_description/meshes/CX165L-J1.STL"/>
+            </geometry>
+            <material
+                name="">
+                <color
+                rgba="0.75294 0.75294 0.75294 1" />
+            </material>
+        </visual>
+        <collision>
+            <origin
+                xyz="0 0 0"
+                rpy="0 0 0" />
+            <geometry>
+                <mesh
+                filename="package://khi_cx_description/meshes/CX165L-J1-HULL.STL" />
             </geometry>
         </collision>
@@ -125,19 +131,19 @@
             <geometry>
                 <mesh
-                filename="package://khi_cx_description/meshes/CX165L-BC01_J2.STL" />
-            </geometry>
-            <material
-                name="">
-                <color
-                rgba="0.75294 0.75294 0.75294 1" />
-            </material>
-        </visual>
-        <collision>
-            <origin
-                xyz="0 0 0"
-                rpy="0 0 0" />
-            <geometry>
-                <mesh
-                filename="package://khi_cx_description/meshes/CX165L-BC01_J2.STL" />
+                filename="package://khi_cx_description/meshes/CX165L-J2.STL" />
+            </geometry>
+            <material
+                name="">
+                <color
+                rgba="0.75294 0.75294 0.75294 1" />
+            </material>
+        </visual>
+        <collision>
+            <origin
+                xyz="0 0 0"
+                rpy="0 0 0" />
+            <geometry>
+                <mesh
+                filename="package://khi_cx_description/meshes/CX165L-J2-HULL.STL" />
             </geometry>
         </collision>
@@ -160,19 +166,19 @@
             <geometry>
                 <mesh
-                filename="package://khi_cx_description/meshes/CX165L-BC01_J3.STL" />
-            </geometry>
-            <material
-                name="">
-                <color
-                rgba="0.75294 0.75294 0.75294 1" />
-            </material>
-        </visual>
-        <collision>
-            <origin
-                xyz="0 0 0"
-                rpy="0 0 0" />
-            <geometry>
-                <mesh
-                filename="package://khi_cx_description/meshes/CX165L-BC01_J3.STL" />
+                filename="package://khi_cx_description/meshes/CX165L-J3.STL" />
+            </geometry>
+            <material
+                name="">
+                <color
+                rgba="0.75294 0.75294 0.75294 1" />
+            </material>
+        </visual>
+        <collision>
+            <origin
+                xyz="0 0 0"
+                rpy="0 0 0" />
+            <geometry>
+                <mesh
+                filename="package://khi_cx_description/meshes/CX165L-J3-HULL.STL" />
             </geometry>
         </collision>
@@ -195,5 +201,5 @@
             <geometry>
                 <mesh
-                filename="package://khi_cx_description/meshes/CX165L-BC01_J4.STL"  />
+                filename="package://khi_cx_description/meshes/CX165L-J4.STL"  />
             </geometry>
             <material
@@ -209,5 +215,5 @@
             <geometry>
                 <mesh
-                filename="package://khi_cx_description/meshes/CX165L-BC01_J4.STL"  />
+                filename="package://khi_cx_description/meshes/CX165L-J4-HULL.STL"  />
             </geometry>
         </collision>
@@ -218,5 +224,5 @@
       <axis xyz="1 0 0" rpy="0 0 0" />
       <limit effort="1000.0" lower="${j5_lower_limit}" upper="${j5_upper_limit}" velocity="${j5_velocity_limit}"/>
-        <origin rpy="0 0 0" xyz="0 0.01 0"/>
+        <origin rpy="0 0 0" xyz="0 0 0"/>
       <parent link="${prefix}link4"/>
       <child link="${prefix}link5"/>
@@ -230,19 +236,19 @@
             <geometry>
                 <mesh
-                filename="package://khi_cx_description/meshes/CX165L-BC01_J5.STL" />
-            </geometry>
-            <material
-                name="">
-                <color
-                rgba="0.75294 0.75294 0.75294 1" />
-            </material>
-        </visual>
-        <collision>
-            <origin
-                xyz="0 0 0"
-                rpy="0 0 0" />
-            <geometry>
-                <mesh
-                filename="package://khi_cx_description/meshes/CX165L-BC01_J5.STL"/>
+                filename="package://khi_cx_description/meshes/CX165L-J5.STL" />
+            </geometry>
+            <material
+                name="">
+                <color
+                rgba="0.75294 0.75294 0.75294 1" />
+            </material>
+        </visual>
+        <collision>
+            <origin
+                xyz="0 0 0"
+                rpy="0 0 0" />
+            <geometry>
+                <mesh
+                filename="package://khi_cx_description/meshes/CX165L-J5-HULL.STL"/>
             </geometry>
         </collision>
@@ -253,5 +259,5 @@
       <axis xyz="0 1 0" rpy="0 0 0" />
       <limit effort="1000.0" lower="${j6_lower_limit}" upper="${j6_upper_limit}" velocity="${j6_velocity_limit}"/>
-      <origin xyz="0 0.225 0" rpy="0 0 0" />
+      <origin xyz="0 0.235 0" rpy="0 0 0" />
       <parent link="${prefix}link5"/>
       <child link="${prefix}link6"/>
@@ -265,19 +271,51 @@
             <geometry>
                 <mesh
-                filename="package://khi_cx_description/meshes/CX165L-BC01_J6.STL" />
-            </geometry>
-            <material
-                name="">
-                <color
-                rgba="0.75294 0.75294 0.75294 1" />
-            </material>
-        </visual>
-        <collision>
-            <origin
-                xyz="0 0 0"
-                rpy="0 0 0" />
-            <geometry>
-                <mesh
-                filename="package://khi_cx_description/meshes/CX165L-BC01_J6.STL" />
+                filename="package://khi_cx_description/meshes/CX165L-J6.STL" />
+            </geometry>
+            <material
+                name="">
+                <color
+                rgba="0.75294 0.75294 0.75294 1" />
+            </material>
+        </visual>
+        <collision>
+            <origin
+                xyz="0 0 0"
+                rpy="0 0 0" />
+            <geometry>
+                <mesh
+                filename="package://khi_cx_description/meshes/CX165L-J6-HULL.STL" />
+            </geometry>
+        </collision>
+        <xacro:default_inertial mass="${j6_mass}"/>
+    </link>
+    <!-- PushCorp Compliant Tool and Spindle -->
+    <joint name="${prefix}pushcorp" type="fixed">
+      <origin xyz="0 0.0949325000000025 0" rpy="0 1.5707963267949 0" />
+      <parent link="${prefix}link6"/>
+      <child link="${prefix}pushcorp"/>
+    </joint>
+    <link name="${prefix}pushcorp">
+        <visual>
+            <origin
+                xyz="0 0 0"
+                rpy="0 0 0" />
+            <geometry>
+                <mesh
+                filename="package://khi_cx_description/meshes/CX165L-PUSHCORP.STL" />
+            </geometry>
+            <material
+                name="">
+                <color
+                rgba="0.75294 0.75294 0.75294 1" />
+            </material>
+        </visual>
+        <collision>
+            <origin
+                xyz="0 0 0"
+                rpy="0 0 0" />
+            <geometry>
+                <mesh
+                filename="package://khi_cx_description/meshes/CX165L-PUSHCORP-HULL.STL" />
             </geometry>
         </collision>

Commit message: updated khi driver

File: khi_cx_description/urdf/cx165l.urdf.xacro (robot description, xacro)
@@ -1,12 +1,12 @@
 <?xml version="1.0" ?>
-<robot name="khi_cx165l" xmlns:xacro="http://ros.org/wiki/xacro">
+<robot name="khi_duaro" xmlns:xacro="http://ros.org/wiki/xacro">
   <xacro:include filename="$(find khi_cx_description)/urdf/cx165l_macro.xacro"/>
-  <!-- instantiate cx165l -->
+  <!-- instantiate duaro -->
   <xacro:khi_cx165l prefix="" />
-  <!-- Fix cx165l to world -->
+  <!-- Fix CX to world -->
   <link name="world"/>
   <joint name="world2base" type="fixed">
     <parent link="world"/>
-    <child link="base_plate"/>
+    <child link="base_link"/>
     <origin rpy="0 0 0" xyz="0 0 0"/>
   </joint>

File: khi_cx_description/urdf/cx165l_macro.xacro (robot description, xacro)
@@ -4,5 +4,4 @@
     <xacro:include filename="$(find khi_cx_description)/urdf/cx.transmission.xacro" />
     <xacro:include filename="$(find khi_cx_description)/urdf/common.gazebo.xacro" />
-    <xacro:include filename="$(find khi_cx_description)/urdf/isu_lab.xacro" />
     <!-- link rviz colors -->
     <material name="White">
@@ -49,5 +48,5 @@
     </xacro:macro>
     <joint name="${prefix}base_link_joint" type="fixed">
-        <parent link="base_plate" />
+        <parent link="world" />
         <child link="base_link" />
         <origin rpy="0 0 0" xyz="0 0 0" />
@@ -117,5 +116,5 @@
     <!-- Link 2 -->
     <joint name="${prefix}joint2" type="revolute">
-      <axis xyz="1 0 0" rpy="0 0 0" />
+      <axis xyz="-1 0 0" rpy="0 0 0" />
       <limit effort="1000.0" lower="${j2_lower_limit}" upper="${j2_upper_limit}" velocity="${j2_velocity_limit}"/>
       <origin xyz="0 0.3 0" rpy="0 0 0" />
@@ -290,36 +289,4 @@
         <xacro:default_inertial mass="${j6_mass}"/>
     </link>
-    <!-- PushCorp Compliant Tool and Spindle -->
-    <joint name="${prefix}pushcorp" type="fixed">
-      <origin xyz="0 0.0949325000000025 0" rpy="0 1.5707963267949 0" />
-      <parent link="${prefix}link6"/>
-      <child link="${prefix}pushcorp"/>
-    </joint>
-    <link name="${prefix}pushcorp">
-        <visual>
-            <origin
-                xyz="0 0 0"
-                rpy="0 0 0" />
-            <geometry>
-                <mesh
-                filename="package://khi_cx_description/meshes/CX165L-PUSHCORP.STL" />
-            </geometry>
-            <material
-                name="">
-                <color
-                rgba="0.75294 0.75294 0.75294 1" />
-            </material>
-        </visual>
-        <collision>
-            <origin
-                xyz="0 0 0"
-                rpy="0 0 0" />
-            <geometry>
-                <mesh
-                filename="package://khi_cx_description/meshes/CX165L-PUSHCORP-HULL.STL" />
-            </geometry>
-        </collision>
-        <xacro:default_inertial mass="${j6_mass}"/>
-    </link>
   </xacro:macro>
 </robot>
